Commit message: using ros2 control to fold the wings

File: src/exocet_mm40b3_description/urdf/exocet_mm40b3.gazebo.xacro (robot description, xacro)
@@ -1,12 +1,6 @@
 <?xml version="1.0" ?>
 <robot name="exocet_mm40b3" xmlns:xacro="http://www.ros.org/wiki/xacro" >
-<gazebo>
-  <plugin name="control" filename="libgazebo_ros_control.so">
-    <robotNamespace>/exocet_mm40b3</robotNamespace>
-    <robotSimType>gazebo_ros_control/DefaultRobotHWSim</robotSimType>
-  </plugin>
-</gazebo>
 <gazebo reference="base_link">
-  <material>Gazebo/Silver</material>
+  <material>Gazebo/White</material>
   <mu1>0.2</mu1>
   <mu2>0.2</mu2>
@@ -87,5 +81,5 @@
 </gazebo>
 <gazebo reference="Booster_1">
-  <material>Gazebo/Silver</material>
+  <material>Gazebo/White</material>
   <mu1>0.2</mu1>
   <mu2>0.2</mu2>
@@ -93,6 +87,6 @@
 </gazebo>
 <gazebo reference="Rigid19">
-  <disableFixedJointLumping>true</disableFixedJointLumping>
-  <preserveFixedJoint>true</preserveFixedJoint>
+  <!-- <disableFixedJointLumping>true</disableFixedJointLumping>  -->
+  <!-- <preserveFixedJoint>true</preserveFixedJoint> -->
 </gazebo>
 </robot>

File: src/exocet_mm40b3_description/urdf/exocet_mm40b3.urdf.xacro (robot description, xacro)
@@ -2,6 +2,7 @@
 <robot name="exocet_mm40b3" xmlns:xacro="http://www.ros.org/wiki/xacro">
 <xacro:include filename="$(find exocet_mm40b3_description)/urdf/materials.xacro" />
-<!-- <xacro:include filename="$(find exocet_mm40b3_description)/urdf/exocet_mm40b3.trans" /> -->
 <xacro:include filename="$(find exocet_mm40b3_description)/urdf/exocet_mm40b3.gazebo.xacro" />
+<xacro:include filename="$(find exocet_mm40b3_description)/urdf/exocet_mm40b3_control.xacro" />
+<xacro:include filename="$(find exocet_mm40b3_description)/urdf/exocet_mm40b3.trans" />
 <link name="base_link">
   <inertial>
@@ -24,5 +25,5 @@
   </collision>
 </link>
-<link name="Fin_1">
+<!-- <link name="Fin_1">
   <inertial>
     <origin xyz="-0.04207063686395979 0.042070952020477254 -0.016310158349904347" rpy="0 0 0"/>
@@ -183,5 +184,5 @@
     </geometry>
   </collision>
-</link>
+</link> -->
 <link name="Wing1_1">
   <inertial>
@@ -284,5 +285,5 @@
   </collision>
 </link>
-<joint name="fins_fold1" type="revolute">
+<!-- <joint name="fins_fold1" type="revolute">
   <origin xyz="-0.04273 0.042755 0.0" rpy="0 0 0"/>
   <parent link="FinHolder_1"/>
@@ -339,5 +340,5 @@
   <axis xyz="0.707107 0.707107 0.0"/>
   <limit upper="0.349066" lower="-0.349066" effort="100" velocity="100"/>
-</joint>
+</joint> -->
 <joint name="wings_fold1" type="revolute">
   <origin xyz="-0.1681 0.1681 2.521299" rpy="0 0 0"/>
